Commit message: remove hard coded file path

File: ur5e_2f_85_description/urdf/ur5e_2f_85.urdf (robot description, URDF)
Before this commit: robot ur5e_2f_85, 22 links, 21 joints
Links:
- link robotiq_85_base_link: geometry collision mesh filename=package://robotiq_description/share/robotiq_description/mes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; visual mesh filename=package://robotiq_description/share/robotiq_description/mes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
- link robotiq_85_left_finger_link: geometry collision mesh filename=package://robotiq_description/share/robotiq_description/mes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; visual mesh filename=package://robotiq_description/share/robotiq_description/mes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
- link robotiq_85_left_finger_tip_link: geometry collision mesh filename=package://robotiq_description/share/robotiq_description/mes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; visual mesh filename=package://robotiq_description/share/robotiq_description/mes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
- link robotiq_85_left_inner_knuckle_link: geometry collision mesh filename=package://robotiq_description/share/robotiq_description/mes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; visual mesh filename=package://robotiq_description/share/robotiq_description/mes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
- link robotiq_85_left_knuckle_link: geometry collision mesh filename=package://robotiq_description/share/robotiq_description/mes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; visual mesh filename=package://robotiq_description/share/robotiq_description/mes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
- link robotiq_85_right_finger_link: geometry collision mesh filename=package://robotiq_description/share/robotiq_description/mes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; visual mesh filename=package://robotiq_description/share/robotiq_description/mes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
- link robotiq_85_right_finger_tip_link: geometry collision mesh filename=package://robotiq_description/share/robotiq_description/mes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; visual mesh filename=package://robotiq_description/share/robotiq_description/mes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
- link robotiq_85_right_inner_knuckle_link: geometry collision mesh filename=package://robotiq_description/share/robotiq_description/mes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; visual mesh filename=package://robotiq_description/share/robotiq_description/mes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
- link robotiq_85_right_knuckle_link: geometry collision mesh filename=package://robotiq_description/share/robotiq_description/mes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; visual mesh filename=package://robotiq_description/share/robotiq_description/mes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
